File: ram.kicad_sch (KiCad schematic)
At the start: 1 part, among them U10 TMM4164AP-15

Commit message: First Draft - RAM
Parts:
- added U11, U12, U13, U14, U15, U16, U17: TMM4164AP-15, Package_DIP:DIP-16_W7.62mm, symbol Laser500:DRAM4164
Connections:
- net MA5: now reaches U10.10 (A5)
- net MA5: now also U11.10 (A5), U12.10 (A5), U13.10 (A5), U14.10 (A5), U15.10 (A5), U16.10 (A5), U17.10 (A5)
- net MA4: now reaches U10.11 (A4)
- net MA4: now also U11.11 (A4), U12.11 (A4), U13.11 (A4), U14.11 (A4), U15.11 (A4), U16.11 (A4), U17.11 (A4)
- net MA3: now reaches U10.12 (A3)
- net MA3: now also U11.12 (A3), U12.12 (A3), U13.12 (A3), U14.12 (A3), U15.12 (A3), U16.12 (A3), U17.12 (A3)
- net MA6: now reaches U10.13 (A6)
- net MA6: now also U11.13 (A6), U12.13 (A6), U13.13 (A6), U14.13 (A6), U15.13 (A6), U16.13 (A6), U17.13 (A6)
- net RD0: now reaches U10.14 (Dout)
- net RD0: now also U10.2 (Din)
- net ~{CAS}: now reaches U10.15 (~{CAS})
- net ~{CAS}: now also U11.15 (~{CAS}), U12.15 (~{CAS}), U13.15 (~{CAS}), U14.15 (~{CAS}), U15.15 (~{CAS}), U16.15 (~{CAS}), U17.15 (~{CAS})
- net ~{RAMW}: now reaches U10.3 (W)
- net ~{RAMW}: now also U11.3 (W), U12.3 (W), U13.3 (W), U14.3 (W), U15.3 (W), U16.3 (W), U17.3 (W)
- net ~{RAS}: now reaches U10.4 (~{RAS})
- net ~{RAS}: now also U11.4 (~{RAS}), U12.4 (~{RAS}), U13.4 (~{RAS}), U14.4 (~{RAS}), U15.4 (~{RAS}), U16.4 (~{RAS}), U17.4 (~{RAS})
- net MA0: now reaches U10.5 (A0)
- net MA0: now also U11.5 (A0), U12.5 (A0), U13.5 (A0), U14.5 (A0), U15.5 (A0), U16.5 (A0), U17.5 (A0)
- net MA2: now reaches U10.6 (A2)
- net MA2: now also U11.6 (A2), U12.6 (A2), U13.6 (A2), U14.6 (A2), U15.6 (A2), U16.6 (A2), U17.6 (A2)
- net MA1: now reaches U10.7 (A1)
- net MA1: now also U11.7 (A1), U12.7 (A1), U13.7 (A1), U14.7 (A1), U15.7 (A1), U16.7 (A1), U17.7 (A1)
- net +5V: now reaches U10.8 (VCC)
- net +5V: now also U11.8 (VCC), U12.8 (VCC), U13.8 (VCC), U14.8 (VCC), U15.8 (VCC), U16.8 (VCC), U17.8 (VCC)
- net MA7: now reaches U10.9 (A7)
- net MA7: now also U11.9 (A7), U12.9 (A7), U13.9 (A7), U14.9 (A7), U15.9 (A7), U16.9 (A7), U17.9 (A7)
- new net RD1: U11.14 (Dout), U11.2 (Din)
- new net RD2: U12.14 (Dout), U12.2 (Din)
- new net RD3: U13.14 (Dout), U13.2 (Din)
- new net RD4: U14.14 (Dout), U14.2 (Din)
- new net RD5: U15.14 (Dout), U15.2 (Din)
- new net RD6: U16.14 (Dout), U16.2 (Din)
- new net RD7: U17.14 (Dout), U17.2 (Din)
Other:
- title: (none) -> Laser 500 4164x8 DRAM
- moved on the sheet: U10

Commit message: Started video_cassette sch
Parts:
- renumbered U10 to U1, U11 to U2, U12 to U3, U13 to U4, U14 to U5, U15 to U6, U16 to U7, U17 to U8
Changed lines of the file:
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@@
 		(dnp no)
 		(fields_autoplaced yes)
-		(property "Reference" "U13"
+		(property "Reference" "U4"
 			(at 144.018 72.136 0)
 			(effects
@@
 			(project "Laser-500"
 				(path "/c1a6b1ae-77c2-4767-93cc-3749547878e9/6122270c-aaa6-4a22-bb6f-62f76c94a913"
-					(reference "U13")
+					(reference "U4")
 					(unit 1)
 				)
@@
 		(dnp no)
 		(fields_autoplaced yes)
-		(property "Reference" "#PWR04"
+		(property "Reference" "#PWR08"
 			(at 154.432 99.314 0)
 			(effects
@@
 			(project "Laser-500"
 				(path "/c1a6b1ae-77c2-4767-93cc-3749547878e9/6122270c-aaa6-4a22-bb6f-62f76c94a913"
-					(reference "#PWR04")
+					(reference "#PWR08")
 					(unit 1)
 				)
@@
 		(dnp no)
 		(fields_autoplaced yes)
-		(property "Reference" "U10"
+		(property "Reference" "U1"
 			(at 51.816 72.136 0)
 			(effects
@@
 			(project ""
 				(path "/c1a6b1ae-77c2-4767-93cc-3749547878e9/6122270c-aaa6-4a22-bb6f-62f76c94a913"
-					(reference "U10")
+					(reference "U1")
 					(unit 1)
 				)
@@
 		(dnp no)
 		(fields_autoplaced yes)
-		(property "Reference" "#PWR07"
+		(property "Reference" "#PWR014"
 			(at 246.888 99.568 0)
 			(effects
@@
 			(project "Laser-500"
 				(path "/c1a6b1ae-77c2-4767-93cc-3749547878e9/6122270c-aaa6-4a22-bb6f-62f76c94a913"
-					(reference "#PWR07")
+					(reference "#PWR014")
 					(unit 1)
 				)
@@
 		(dnp no)
 		(fields_autoplaced yes)
-		(property "Reference" "U14"
+		(property "Reference" "U5"
 			(at 174.244 72.136 0)
 			(effects
@@
 			(project "Laser-500"
 				(path "/c1a6b1ae-77c2-4767-93cc-3749547878e9/6122270c-aaa6-4a22-bb6f-62f76c94a913"
-					(reference "U14")
+					(reference "U5")
 					(unit 1)
 				)
@@
 		(dnp no)
 		(fields_autoplaced yes)
-		(property "Reference" "#PWR01"
+		(property "Reference" "#PWR02"
 			(at 62.484 99.568 0)
 			(effects
@@
 			(project ""
 				(path "/c1a6b1ae-77c2-4767-93cc-3749547878e9/6122270c-aaa6-4a22-bb6f-62f76c94a913"
-					(reference "#PWR01")
+					(reference "#PWR02")
 					(unit 1)
 				)
@@
 		(on_board yes)
 		(dnp no)
-		(property "Reference" "#PWR09"
+		(property "Reference" "#PWR01"
 			(at 62.484 91.948 0)
 			(effects
@@
 			(project ""
 				(path "/c1a6b1ae-77c2-4767-93cc-3749547878e9/6122270c-aaa6-4a22-bb6f-62f76c94a913"
-					(reference "#PWR09")
+					(reference "#PWR01")
 					(unit 1)
 				)
@@
 		(on_board yes)
 		(dnp no)
-		(property "Reference" "#PWR011"
+		(property "Reference" "#PWR05"
 			(at 123.444 92.202 0)
 			(effects
@@
 			(project "Laser-500"
 				(path "/c1a6b1ae-77c2-4767-93cc-3749547878e9/6122270c-aaa6-4a22-bb6f-62f76c94a913"
-					(reference "#PWR011")
+					(reference "#PWR05")
 					(unit 1)
 				)
@@
 		(dnp no)
 		(fields_autoplaced yes)
-		(property "Reference" "U17"
+		(property "Reference" "U8"
 			(at 266.954 72.39 0)
 			(effects
@@
 			(project "Laser-500"
 				(path "/c1a6b1ae-77c2-4767-93cc-3749547878e9/6122270c-aaa6-4a22-bb6f-62f76c94a913"
-					(reference "U17")
+					(reference "U8")
 					(unit 1)
 				)
@@
 		(on_board yes)
 		(dnp no)
-		(property "Reference" "#PWR010"
+		(property "Reference" "#PWR03"
 			(at 93.472 91.948 0)
 			(effects
@@
 			(project "Laser-500"
 				(path "/c1a6b1ae-77c2-4767-93cc-3749547878e9/6122270c-aaa6-4a22-bb6f-62f76c94a913"
-					(reference "#PWR010")
+					(reference "#PWR03")
 					(unit 1)
 				)
@@
 		(dnp no)
 		(fields_autoplaced yes)
-		(property "Reference" "U11"
+		(property "Reference" "U2"
 			(at 82.804 72.136 0)
 			(effects
@@
 			(project "Laser-500"
 				(path "/c1a6b1ae-77c2-4767-93cc-3749547878e9/6122270c-aaa6-4a22-bb6f-62f76c94a913"
-					(reference "U11")
+					(reference "U2")
 					(unit 1)
 				)
@@
 		(dnp no)
 		(fields_autoplaced yes)
-		(property "Reference" "U15"
+		(property "Reference" "U6"
 			(at 205.232 72.136 0)
 			(effects
@@
 			(project "Laser-500"
 				(path "/c1a6b1ae-77c2-4767-93cc-3749547878e9/6122270c-aaa6-4a22-bb6f-62f76c94a913"
-					(reference "U15")
+					(reference "U6")
 					(unit 1)
 				)
@@
 		(dnp no)
 		(fields_autoplaced yes)
-		(property "Reference" "#PWR06"
+		(property "Reference" "#PWR012"
 			(at 215.9 99.314 0)
 			(effects
@@
 			(project "Laser-500"
 				(path "/c1a6b1ae-77c2-4767-93cc-3749547878e9/6122270c-aaa6-4a22-bb6f-62f76c94a913"
-					(reference "#PWR06")
+					(reference "#PWR012")
 					(unit 1)
 				)
@@
 		(dnp no)
 		(fields_autoplaced yes)
-		(property "Reference" "#PWR03"
+		(property "Reference" "#PWR06"
 			(at 123.444 99.822 0)
 			(effects
@@
 			(project "Laser-500"
 				(path "/c1a6b1ae-77c2-4767-93cc-3749547878e9/6122270c-aaa6-4a22-bb6f-62f76c94a913"
-					(reference "#PWR03")
+					(reference "#PWR06")
 					(unit 1)
 				)
@@
 		(dnp no)
 		(fields_autoplaced yes)
-		(property "Reference" "#PWR02"
+		(property "Reference" "#PWR04"
 			(at 93.472 99.568 0)
 			(effects
@@
 			(project "Laser-500"
 				(path "/c1a6b1ae-77c2-4767-93cc-3749547878e9/6122270c-aaa6-4a22-bb6f-62f76c94a913"
-					(reference "#PWR02")
+					(reference "#PWR04")
 					(unit 1)
 				)
@@
 		(dnp no)
 		(fields_autoplaced yes)
-		(property "Reference" "U12"
+		(property "Reference" "U3"
 			(at 113.284 72.136 0)
 			(effects
@@
 			(project "Laser-500"
 				(path "/c1a6b1ae-77c2-4767-93cc-3749547878e9/6122270c-aaa6-4a22-bb6f-62f76c94a913"
-					(reference "U12")
+					(reference "U3")
 					(unit 1)
 				)
@@
 		(on_board yes)
 		(dnp no)
-		(property "Reference" "#PWR012"
+		(property "Reference" "#PWR07"
 			(at 154.432 92.202 0)
 			(effects
@@
 			(project "Laser-500"
 				(path "/c1a6b1ae-77c2-4767-93cc-3749547878e9/6122270c-aaa6-4a22-bb6f-62f76c94a913"
-					(reference "#PWR012")
+					(reference "#PWR07")
 					(unit 1)
 				)
@@
 		(dnp no)
 		(fields_autoplaced yes)
-		(property "Reference" "#PWR05"
+		(property "Reference" "#PWR010"
 			(at 185.166 99.314 0)
 			(effects
@@
 			(project "Laser-500"
 				(path "/c1a6b1ae-77c2-4767-93cc-3749547878e9/6122270c-aaa6-4a22-bb6f-62f76c94a913"
-					(reference "#PWR05")
+					(reference "#PWR010")
 					(unit 1)
 				)
@@
 		(on_board yes)
 		(dnp no)
-		(property "Reference" "#PWR015"
+		(property "Reference" "#PWR013"
 			(at 246.888 92.456 0)
 			(effects
@@
 			(project "Laser-500"
 				(path "/c1a6b1ae-77c2-4767-93cc-3749547878e9/6122270c-aaa6-4a22-bb6f-62f76c94a913"
-					(reference "#PWR015")
+					(reference "#PWR013")
 					(unit 1)
 				)
@@
 		(on_board yes)
 		(dnp no)
-		(property "Reference" "#PWR016"
+		(property "Reference" "#PWR015"
 			(at 278.892 92.202 0)
 			(effects
@@
 			(project "Laser-500"
 				(path "/c1a6b1ae-77c2-4767-93cc-3749547878e9/6122270c-aaa6-4a22-bb6f-62f76c94a913"
-					(reference "#PWR016")
+					(reference "#PWR015")
 					(unit 1)
 				)
@@
 		(on_board yes)
 		(dnp no)
-		(property "Reference" "#PWR013"
+		(property "Reference" "#PWR09"
 			(at 185.166 92.202 0)
 			(effects
@@
 			(project "Laser-500"
 				(path "/c1a6b1ae-77c2-4767-93cc-3749547878e9/6122270c-aaa6-4a22-bb6f-62f76c94a913"
-					(reference "#PWR013")
+					(reference "#PWR09")
 					(unit 1)
 				)
@@
 		(dnp no)
 		(fields_autoplaced yes)
-		(property "Reference" "U16"
+		(property "Reference" "U7"
 			(at 235.966 72.39 0)
 			(effects
@@
 			(project "Laser-500"
 				(path "/c1a6b1ae-77c2-4767-93cc-3749547878e9/6122270c-aaa6-4a22-bb6f-62f76c94a913"
-					(reference "U16")
+					(reference "U7")
 					(unit 1)
 				)
@@
 		(on_board yes)
 		(dnp no)
-		(property "Reference" "#PWR014"
+		(property "Reference" "#PWR011"
 			(at 215.9 92.456 0)
 			(effects
@@
 			(project "Laser-500"
 				(path "/c1a6b1ae-77c2-4767-93cc-3749547878e9/6122270c-aaa6-4a22-bb6f-62f76c94a913"
-					(reference "#PWR014")
+					(reference "#PWR011")
 					(unit 1)
 				)
@@
 		(dnp no)
 		(fields_autoplaced yes)
-		(property "Reference" "#PWR08"
+		(property "Reference" "#PWR016"
 			(at 278.892 100.584 0)
 			(effects
@@
 			(project "Laser-500"
 				(path "/c1a6b1ae-77c2-4767-93cc-3749547878e9/6122270c-aaa6-4a22-bb6f-62f76c94a913"
-					(reference "#PWR08")
-					(unit 1)
-				)
+					(reference "#PWR016")
+					(unit 1)
+				)

Commit message: Finished Y-signal generation
Changed lines of the file:
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@@
 	)
 	(junction
-		(at 19.304 110.744)
-		(diameter 0)
-		(color 0 0 0 0)
-	)
-	(junction
 		(at 224.282 110.744)
 		(diameter 0)
@@
 	)
 	(junction
-		(at 19.558 123.444)
-		(diameter 0)
-		(color 0 0 0 0)
-	)
-	(junction
 		(at 123.698 81.534)
 		(diameter 0)
@@
 	)
 	(junction
-		(at 19.558 51.816)
-		(diameter 0)
-		(color 0 0 0 0)
-	)
-	(junction
 		(at 39.37 110.744)
 		(diameter 0)
@@
 	)
 	(junction
-		(at 19.812 60.452)
-		(diameter 0)
-		(color 0 0 0 0)
-	)
-	(junction
 		(at 244.856 81.788)
 		(diameter 0)
@@
 	)
 	(junction
-		(at 19.304 116.332)
-		(diameter 0)
-		(color 0 0 0 0)
-	)
-	(junction
 		(at 103.378 116.332)
 		(diameter 0)
@@
 	(wire
 		(pts
-			(xy 19.304 116.332) (xy 41.402 116.332)
-		)
-		(stroke
-			(width 0)
-			(type default)
-		)
-	)
-	(wire
-		(pts
 			(xy 192.532 89.154) (xy 196.342 89.154)
 		)
@@
 	(bus
 		(pts
-			(xy 16.764 60.452) (xy 19.812 60.452)
+			(xy 27.432 60.452) (xy 34.544 60.452)
 		)
 		(stroke
@@
 	(wire
 		(pts
-			(xy 16.764 116.332) (xy 19.304 116.332)
+			(xy 24.892 116.332) (xy 41.402 116.332)
 		)
 		(stroke
@@
 	(wire
 		(pts
-			(xy 19.304 113.792) (xy 19.304 116.332)
-		)
-		(stroke
-			(width 0)
-			(type default)
-		)
-	)
-	(wire
-		(pts
 			(xy 93.98 99.314) (xy 93.98 123.444)
 		)
@@
 	(wire
 		(pts
-			(xy 19.558 123.444) (xy 62.992 123.444)
+			(xy 23.114 123.444) (xy 62.992 123.444)
 		)
 		(stroke
@@
 	(wire
 		(pts
-			(xy 19.304 107.95) (xy 19.304 110.744)
-		)
-		(stroke
-			(width 0)
-			(type default)
-		)
-	)
-	(wire
-		(pts
 			(xy 152.908 91.694) (xy 154.432 91.694)
 		)
@@
 		)
 	)
-	(bus
-		(pts
-			(xy 19.812 56.896) (xy 19.812 60.452)
-		)
-		(stroke
-			(width 0)
-			(type default)
-		)
-	)
 	(wire
 		(pts
@@
 		)
 	)
-	(bus
-		(pts
-			(xy 19.558 49.022) (xy 19.558 51.816)
-		)
-		(stroke
-			(width 0)
-			(type default)
-		)
-	)
 	(wire
 		(pts
@@
 	(bus
 		(pts
-			(xy 16.764 51.816) (xy 19.558 51.816)
+			(xy 27.432 51.816) (xy 59.69 51.816)
 		)
 		(stroke
@@
 		)
 	)
-	(bus
-		(pts
-			(xy 19.812 60.452) (xy 34.544 60.452)
-		)
-		(stroke
-			(width 0)
-			(type default)
-		)
-	)
 	(wire
 		(pts
@@
 	(wire
 		(pts
-			(xy 16.764 110.744) (xy 19.304 110.744)
+			(xy 23.114 110.744) (xy 39.37 110.744)
 		)
 		(stroke
@@
 	(bus
 		(pts
-			(xy 19.558 51.816) (xy 59.69 51.816)
-		)
-		(stroke
-			(width 0)
-			(type default)
-		)
-	)
-	(bus
-		(pts
 			(xy 189.992 81.534) (xy 189.992 78.994)
 		)
@@
 	(wire
 		(pts
-			(xy 16.764 123.444) (xy 19.558 123.444)
-		)
-		(stroke
-			(width 0)
-			(type default)
-		)
-	)
-	(wire
-		(pts
 			(xy 123.444 88.392) (xy 123.444 89.154)
 		)
@@
 	(wire
 		(pts
-			(xy 19.558 120.65) (xy 19.558 123.444)
-		)
-		(stroke
-			(width 0)
-			(type default)
-		)
-	)
-	(wire
-		(pts
 			(xy 225.806 116.332) (xy 256.794 116.332)
 		)
@@
 	(wire
 		(pts
-			(xy 19.304 110.744) (xy 39.37 110.744)
-		)
-		(stroke
-			(width 0)
-			(type default)
-		)
-	)
-	(wire
-		(pts
 			(xy 215.646 54.356) (xy 215.646 81.534)
 		)
@@
 		)
 	)
-	(global_label "MA[0..7]"
+	(global_label "~{RAS}"
 		(shape input)
-		(at 19.812 56.896 0)
+		(at 23.114 110.744 180)
 		(fields_autoplaced yes)
 		(effects
@@
 				(size 1.27 1.27)
 			)
-			(justify left)
+			(justify right)
 		)
 		(property "Intersheetrefs" "${INTERSHEET_REFS}"
-			(at 30.6592 56.896 0)
+			(at 16.5607 110.744 0)
 			(effects
 				(font
 					(size 1.27 1.27)
 				)
-				(justify left)
+				(justify right)
 				(hide yes)
 			)
 		)
 	)
-	(global_label "RD[0..7]"
-		(shape bidirectional)
-		(at 19.558 49.022 0)
+	(global_label "~{RAMW}"
+		(shape input)
+		(at 24.892 116.332 180)
 		(fields_autoplaced yes)
 		(effects
@@
 				(size 1.27 1.27)
 			)
-			(justify left)
+			(justify right)
 		)
 		(property "Intersheetrefs" "${INTERSHEET_REFS}"
-			(at 31.5165 49.022 0)
+			(at 16.6454 116.332 0)
 			(effects
 				(font
 					(size 1.27 1.27)
 				)
-				(justify left)
+				(justify right)
 				(hide yes)
 			)
 		)
 	)
-	(global_label "~{RAMW}"
-		(shape output)
-		(at 19.304 113.792 0)
+	(global_label "~{CAS}"
+		(shape input)
+		(at 23.114 123.444 180)
 		(fields_autoplaced yes)
 		(effects
@@
 				(size 1.27 1.27)
 			)
-			(justify left)
+			(justify right)
 		)
 		(property "Intersheetrefs" "${INTERSHEET_REFS}"
-			(at 27.5506 113.792 0)
+			(at 16.5607 123.444 0)
 			(effects
 				(font
 					(size 1.27 1.27)
 				)
-				(justify left)
+				(justify right)
 				(hide yes)
 			)
 		)
 	)
-	(global_label "~{CAS}"
-		(shape output)
-		(at 19.558 120.65 0)
+	(global_label "MA[0..7]"
+		(shape input)
+		(at 27.432 60.452 180)
 		(fields_autoplaced yes)
 		(effects
@@
 				(size 1.27 1.27)
 			)
-			(justify left)
+			(justify right)
 		)
 		(property "Intersheetrefs" "${INTERSHEET_REFS}"
-			(at 26.1113 120.65 0)
+			(at 16.5848 60.452 0)
 			(effects
 				(font
 					(size 1.27 1.27)
 				)
-				(justify left)
+				(justify right)
 				(hide yes)
 			)
 		)
 	)
-	(global_label "~{RAS}"
-		(shape output)
-		(at 19.304 107.95 0)
+	(global_label "RD[0..7]"
+		(shape input)
+		(at 27.432 51.816 180)
 		(fields_autoplaced yes)
 		(effects
@@
 				(size 1.27 1.27)
 			)
-			(justify left)
+			(justify right)
 		)
 		(property "Intersheetrefs" "${INTERSHEET_REFS}"
-			(at 25.8573 107.95 0)
+			(at 16.5848 51.816 0)
 			(effects
 				(font
 					(size 1.27 1.27)
 				)
-				(justify left)
+				(justify right)
 				(hide yes)
 			)

Commit message: A few Boxing day updates
1. Add Laser 500 Mainboard PCB photo
2. Updated Main circuit ICs and their symbols.
3. Updated references according to PCB photo
Parts:
- renumbered U1 to U11, U2 to U12, U3 to U13, U4 to U14, U5 to U15, U6 to U16, U7 to U17, U8 to U18
Changed lines of the file:
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@@
 		(dnp no)
 		(fields_autoplaced yes)
-		(property "Reference" "U4"
+		(property "Reference" "U14"
 			(at 144.018 72.136 0)
 			(effects
@@
 			(project "Laser-500"
 				(path "/c1a6b1ae-77c2-4767-93cc-3749547878e9/6122270c-aaa6-4a22-bb6f-62f76c94a913"
-					(reference "U4")
+					(reference "U14")
 					(unit 1)
 				)
@@
 		(dnp no)
 		(fields_autoplaced yes)
-		(property "Reference" "U1"
+		(property "Reference" "U11"
 			(at 51.816 72.136 0)
 			(effects
@@
 			(project ""
 				(path "/c1a6b1ae-77c2-4767-93cc-3749547878e9/6122270c-aaa6-4a22-bb6f-62f76c94a913"
-					(reference "U1")
+					(reference "U11")
 					(unit 1)
 				)
@@
 		(dnp no)
 		(fields_autoplaced yes)
-		(property "Reference" "U5"
+		(property "Reference" "U15"
 			(at 174.244 72.136 0)
 			(effects
@@
 			(project "Laser-500"
 				(path "/c1a6b1ae-77c2-4767-93cc-3749547878e9/6122270c-aaa6-4a22-bb6f-62f76c94a913"
-					(reference "U5")
+					(reference "U15")
 					(unit 1)
 				)
@@
 		(dnp no)
 		(fields_autoplaced yes)
-		(property "Reference" "U8"
+		(property "Reference" "U18"
 			(at 266.954 72.39 0)
 			(effects
@@
 			(project "Laser-500"
 				(path "/c1a6b1ae-77c2-4767-93cc-3749547878e9/6122270c-aaa6-4a22-bb6f-62f76c94a913"
-					(reference "U8")
+					(reference "U18")
 					(unit 1)
 				)
@@
 		(dnp no)
 		(fields_autoplaced yes)
-		(property "Reference" "U2"
+		(property "Reference" "U12"
 			(at 82.804 72.136 0)
 			(effects
@@
 			(project "Laser-500"
 				(path "/c1a6b1ae-77c2-4767-93cc-3749547878e9/6122270c-aaa6-4a22-bb6f-62f76c94a913"
-					(reference "U2")
+					(reference "U12")
 					(unit 1)
 				)
@@
 		(dnp no)
 		(fields_autoplaced yes)
-		(property "Reference" "U6"
+		(property "Reference" "U16"
 			(at 205.232 72.136 0)
 			(effects
@@
 			(project "Laser-500"
 				(path "/c1a6b1ae-77c2-4767-93cc-3749547878e9/6122270c-aaa6-4a22-bb6f-62f76c94a913"
-					(reference "U6")
+					(reference "U16")
 					(unit 1)
 				)
@@
 		(dnp no)
 		(fields_autoplaced yes)
-		(property "Reference" "U3"
+		(property "Reference" "U13"
 			(at 113.284 72.136 0)
 			(effects
@@
 			(project "Laser-500"
 				(path "/c1a6b1ae-77c2-4767-93cc-3749547878e9/6122270c-aaa6-4a22-bb6f-62f76c94a913"
-					(reference "U3")
+					(reference "U13")
 					(unit 1)
 				)
@@
 		(dnp no)
 		(fields_autoplaced yes)
-		(property "Reference" "U7"
+		(property "Reference" "U17"
 			(at 235.966 72.39 0)
 			(effects
@@
 			(project "Laser-500"
 				(path "/c1a6b1ae-77c2-4767-93cc-3749547878e9/6122270c-aaa6-4a22-bb6f-62f76c94a913"
-					(reference "U7")
-					(unit 1)
-				)
+					(reference "U17")
+					(unit 1)
+				)

Commit message: Started A[0..15] and MA[0..7] on main circuit
Changed lines of the file:
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@@
 	)
 	(bus_entry
-		(at 90.678 51.816)
+		(at 36.576 91.694)
 		(size 2.54 2.54)
 		(stroke
@@
 	)
 	(bus_entry
-		(at 98.044 84.074)
+		(at 90.678 51.816)
 		(size 2.54 2.54)
 		(stroke
@@
 	)
 	(bus_entry
-		(at 67.564 76.454)
+		(at 98.044 84.074)
 		(size 2.54 2.54)
 		(stroke
@@
 	)
 	(bus_entry
-		(at 242.316 51.816)
+		(at 67.564 76.454)
 		(size 2.54 2.54)
 		(stroke
@@
 	)
 	(bus_entry
-		(at 98.044 94.234)
+		(at 242.316 51.816)
 		(size 2.54 2.54)
 		(stroke
@@
 	)
 	(bus_entry
-		(at 159.004 84.074)
+		(at 98.044 94.234)
 		(size 2.54 2.54)
 		(stroke
@@
 	)
 	(bus_entry
-		(at 59.69 51.816)
+		(at 159.004 84.074)
 		(size 2.54 2.54)
 		(stroke
@@
 	)
 	(bus_entry
-		(at 36.576 91.694)
+		(at 59.69 51.816)
 		(size 2.54 2.54)
 		(stroke
@@
 	(bus
 		(pts
-			(xy 36.576 91.694) (xy 36.576 89.154)
-		)
-		(stroke
-			(width 0)
-			(type default)
-		)
-	)
-	(bus
-		(pts
 			(xy 128.778 94.234) (xy 128.778 91.694)
 		)
@@
 		)
 	)
+	(bus
+		(pts
+			(xy 36.576 91.694) (xy 36.576 94.234)
+		)
+		(stroke
+			(width 0)
+			(type default)
+		)
+	)
 	(wire
 		(pts
@@
 	(wire
 		(pts
+			(xy 39.116 94.234) (xy 42.926 94.234)
+		)
+		(stroke
+			(width 0)
+			(type default)
+		)
+	)
+	(wire
+		(pts
 			(xy 225.806 116.332) (xy 256.794 116.332)
 		)
@@
 		)
 	)
-	(wire
-		(pts
-			(xy 39.116 94.234) (xy 42.926 94.234)
-		)
-		(stroke
-			(width 0)
-			(type default)
-		)
-	)
 	(bus
 		(pts
@@
 	(bus
 		(pts
-			(xy 36.576 94.234) (xy 36.576 91.694)
+			(xy 36.576 89.154) (xy 36.576 91.694)
 		)
 		(stroke
@@
 		)
 	)
-	(label "MA1"
-		(at 39.116 94.234 0)
-		(fields_autoplaced yes)
-		(effects
-			(font
-				(size 1.27 1.27)
-			)
-			(justify left bottom)
-		)
-	)
 	(label "MA5"
 		(at 70.104 84.074 0)
@@
 		(fields_autoplaced yes)
 		(effects
+			(font
+				(size 1.27 1.27)
+			)
+			(justify left bottom)
+		)
+	)
+	(label "MA1"
+		(at 39.116 94.234 0)
+		(fields_autoplaced yes)
+		(effects
